File: hw/picoballoon.kicad_pcb (KiCad board)
At the start: 2 copper layers, 51.2 x 20 mm, 30 parts, among them J1 Conn_ARM_JTAG_SWD_10, J4 u.fl, U1 TPS610994YFFR, U2 K32L2B21VLH0A, U3 L96-M33, U4 INNOCOMM-SN10-11, U5 MS561101BA03-50

Commit message: gnss_uart
Parts:
- removed R3, R4: 10k, Resistor_SMD:R_0603_1608Metric
Connections:
- U2 pad 39: unconnected-(U2-PTB16-Pad39) -> /GNSS_TX
- U2 pad 40: unconnected-(U2-PTB17-Pad40) -> /GNSS_RX
- U2 pad 44: /GNSS_I2C_SCL -> unconnected-(U2-PTC1/LLWU_P6/RTC_CLKIN-Pad44)
- U2 pad 45: /GNSS_I2C_SDA -> unconnected-(U2-PTC2-Pad45)
- U3 pad 25: unconnected-(U3-TXD1-Pad25) -> /GNSS_TX
- U3 pad 26: unconnected-(U3-RXD1-Pad26) -> /GNSS_RX
- U3 pad 3: /GNSS_I2C_SDA -> unconnected-(U3-I2C_SDA-Pad3)
- U3 pad 6: /GNSS_I2C_SCL -> unconnected-(U3-I2C_SCL-Pad6)
Routing:
- net /GNSS_TX: track 0.00 -> 24.3 mm, vias 0 -> 1
- net /GNSS_RX: track 0.00 -> 19.1 mm, vias 0 -> 1
- net /GNSS_I2C_SCL: track 13.4 -> 0.00 mm, vias 1 -> 0
- net /GNSS_I2C_SDA: track 10.2 -> 0.00 mm, vias 1 -> 0
- net +3V3: track 88.1 -> 85.3 mm, vias 5 -> 4
