File: hw/picoballoon.kicad_sch (KiCad schematic)
At the start: 29 parts, among them J1 Conn_ARM_JTAG_SWD_10, J2 Conn_01x01, J3 Conn_01x01, J4 u.fl, U1 TPS610994YFFR, U2 K32L2B21VLH0A, U3 L96-M33, U4 INNOCOMM-SN10-11, U5 MS561101BA03-50

Commit message: part #s
Parts:
- C1, C10, C2, C4: Manufacturer_Part_Number (none) -> JMK107ABJ106MA-T
- C11, C15, C20, C5, C6, C8, C9: Manufacturer_Part_Number (none) -> CL10B104KO8NNWC
- C12: Manufacturer_Part_Number (none) -> CL10A475KQ8NNNC; Mouser Part Number (none) -> CL10A475KQ8NNNC
- C13: Manufacturer_Part_Number (none) -> GRM188R60G476ME15J; Mouser Part Number (none) -> GRM188R60G476ME15J
- C14, C7: Manufacturer_Part_Number (none) -> CL10C330JC81PNC
- J1: Manufacturer_Part_Number (none) -> M50-3500542
- J2, J3: Manufacturer_Part_Number (none) -> dnp
- J4: Manufacturer_Part_Number (none) -> 73412-0110
- L1: Manufacturer_Part_Number (none) -> LQM18PN2R2MGHD
- R2: Manufacturer_Part_Number (none) -> RC0603FR-0730RL; Mouser Part Number (none) -> RC0603FR-0730RL
- R3, R4, R5: Manufacturer_Part_Number (none) -> RC0603JR-0710KP
- U1: Manufacturer_Part_Number (none) -> TPS610994YFFR
- U2: Manufacturer_Part_Number (none) -> K32L2B21VLH0A
- U3: Manufacturer_Part_Number (none) -> L96-M33
- U4: Manufacturer_Part_Number (none) -> INNOCOMM-SN10-11
Changed lines of the file:
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@@
+      (effects (font (size 1.27 1.27)) hide)
+    )
+    (property "Manufacturer_Part_Number" "CL10B104KO8NNWC" (at 67.31 101.6 0)
       (effects (font (size 1.27 1.27)) hide)
     )
@@
       (effects (font (size 1.27 1.27)) hide)
     )
+    (property "Manufacturer_Part_Number" "RC0603JR-0710KP" (at 193.04 71.12 0)
+      (effects (font (size 1.27 1.27)) hide)
+    )
     (pin "1")
     (pin "2")
@@
     (property "Datasheet" "https://www.nxp.com/products/processors-and-microcontrollers/arm-microcontrollers/general-purpose-mcus/k32-l-series-cortex-m4-m0-plus/k32-l2-ultra-low-power-highly-integrated-mcu:K32-L2?tab=Documentation_Tab" (at 115.57 167.64 0)
       (effects (font (size 1.27 1.27)) (justify left bottom) hide)
+    )
+    (property "Manufacturer_Part_Number" "K32L2B21VLH0A" (at 107.95 111.76 0)
+      (effects (font (size 1.27 1.27)) hide)
     )
     (pin "1")
@@
       (effects (font (size 1.27 1.27)) hide)
     )
+    (property "Manufacturer_Part_Number" "INNOCOMM-SN10-11" (at 241.3 100.33 0)
+      (effects (font (size 1.27 1.27)) hide)
+    )
     (pin "1")
     (pin "10")
@@
       (effects (font (size 1.27 1.27)) hide)
     )
+    (property "Manufacturer_Part_Number" "73412-0110" (at 274.32 92.71 0)
+      (effects (font (size 1.27 1.27)) hide)
+    )
     (pin "1")
     (pin "2")
@@
       (effects (font (size 1.27 1.27)) hide)
     )
+    (property "Manufacturer_Part_Number" "CL10B104KO8NNWC" (at 137.16 52.07 0)
+      (effects (font (size 1.27 1.27)) hide)
+    )
     (pin "1")
     (pin "2")
@@
       (effects (font (size 1.27 1.27)) hide)
     )
+    (property "Manufacturer_Part_Number" "RC0603JR-0710KP" (at 185.42 71.12 0)
+      (effects (font (size 1.27 1.27)) hide)
+    )
     (pin "1")
     (pin "2")
@@
       (effects (font (size 1.27 1.27)) hide)
     )
+    (property "Manufacturer_Part_Number" "CL10B104KO8NNWC" (at 209.55 55.88 0)
+      (effects (font (size 1.27 1.27)) hide)
+    )
     (pin "1")
     (pin "2")
@@
     )
     (property "Datasheet" "~" (at 266.7 142.24 0)
+      (effects (font (size 1.27 1.27)) hide)
+    )
+    (property "Manufacturer_Part_Number" "CL10B104KO8NNWC" (at 266.7 142.24 0)
       (effects (font (size 1.27 1.27)) hide)
     )
@@
       (effects (font (size 1.27 1.27)) hide)
     )
+    (property "Manufacturer_Part_Number" "dnp" (at 30.48 78.74 0)
+      (effects (font (size 1.27 1.27)) hide)
+    )
     (pin "1")
     (instances
@@
     )
     (property "Datasheet" "~" (at 147.32 52.07 0)
+      (effects (font (size 1.27 1.27)) hide)
+    )
+    (property "Manufacturer_Part_Number" "CL10B104KO8NNWC" (at 147.32 52.07 0)
       (effects (font (size 1.27 1.27)) hide)
     )
@@
       (effects (font (size 1.27 1.27)) hide)
     )
+    (property "Manufacturer_Part_Number" "JMK107ABJ106MA-T " (at 186.69 46.99 0)
+      (effects (font (size 1.27 1.27)) hide)
+    )
     (pin "1")
     (pin "2")
@@
       (effects (font (size 1.27 1.27)) hide)
     )
+    (property "Manufacturer_Part_Number" "GRM188R60G476ME15J" (at 247.65 68.58 0)
+      (effects (font (size 1.27 1.27)) hide)
+    )
+    (property "Mouser Part Number" "GRM188R60G476ME15J" (at 247.65 68.58 0)
+      (effects (font (size 1.27 1.27)) hide)
+    )
     (pin "1")
     (pin "2")
@@
       (effects (font (size 1.27 1.27)) hide)
     )
+    (property "Manufacturer_Part_Number" "CL10C330JC81PNC" (at 247.65 77.47 0)
+      (effects (font (size 1.27 1.27)) hide)
+    )
     (pin "1")
     (pin "2")
@@
     )
     (property "Datasheet" "~" (at 144.78 154.94 0)
+      (effects (font (size 1.27 1.27)) hide)
+    )
+    (property "Manufacturer_Part_Number" "CL10C330JC81PNC" (at 144.78 154.94 0)
       (effects (font (size 1.27 1.27)) hide)
     )
@@
     (property "Datasheet" "https://www.ti.com/lit/ds/symlink/tps61099.pdf" (at 38.1 36.83 0)
       (effects (font (size 1.524 1.524)) hide)
+    )
+    (property "Manufacturer_Part_Number" "TPS610994YFFR" (at 38.1 36.83 0)
+      (effects (font (size 1.27 1.27)) hide)
     )
     (pin "A1")
@@
       (effects (font (size 1.27 1.27)) hide)
     )
+    (property "Manufacturer_Part_Number" "RC0603JR-0710KP" (at 67.31 91.44 0)
+      (effects (font (size 1.27 1.27)) hide)
+    )
     (pin "1")
     (pin "2")
@@
       (effects (font (size 1.27 1.27)) hide)
     )
+    (property "Manufacturer_Part_Number" "JMK107ABJ106MA-T " (at 55.88 39.37 0)
+      (effects (font (size 1.27 1.27)) hide)
+    )
     (pin "1")
     (pin "2")
@@
     )
     (property "Datasheet" "" (at 191.77 22.86 0)
+      (effects (font (size 1.27 1.27)) hide)
+    )
+    (property "Manufacturer_Part_Number" "L96-M33" (at 209.55 38.1 0)
       (effects (font (size 1.27 1.27)) hide)
     )
@@
       (effects (font (size 1.27 1.27)) hide)
     )
+    (property "Manufacturer_Part_Number" "RC0603FR-0730RL" (at 144.78 144.78 0)
+      (effects (font (size 1.27 1.27)) hide)
+    )
+    (property "Mouser Part Number" "RC0603FR-0730RL" (at 144.78 144.78 0)
+      (effects (font (size 1.27 1.27)) hide)
+    )
     (pin "1")
     (pin "2")
@@
       (effects (font (size 1.27 1.27)) hide)
     )
+    (property "Manufacturer_Part_Number" "CL10B104KO8NNWC" (at 127 52.07 0)
+      (effects (font (size 1.27 1.27)) hide)
+    )
     (pin "1")
     (pin "2")
@@
       (effects (font (size 1.27 1.27)) hide)
     )
+    (property "Manufacturer_Part_Number" "CL10A475KQ8NNNC " (at 209.55 64.77 0)
+      (effects (font (size 1.27 1.27)) hide)
+    )
+    (property "Mouser Part Number" "CL10A475KQ8NNNC" (at 209.55 64.77 0)
+      (effects (font (size 1.27 1.27)) hide)
+    )
     (pin "1")
     (pin "2")
@@
     )
     (property "Datasheet" "~" (at 19.05 39.37 0)
+      (effects (font (size 1.27 1.27)) hide)
+    )
+    (property "Manufacturer_Part_Number" "JMK107ABJ106MA-T " (at 19.05 39.37 0)
       (effects (font (size 1.27 1.27)) hide)
     )
@@
     )
     (property "Datasheet" "~" (at 176.53 46.99 0)
+      (effects (font (size 1.27 1.27)) hide)
+    )
+    (property "Manufacturer_Part_Number" "CL10B104KO8NNWC" (at 176.53 46.99 0)
       (effects (font (size 1.27 1.27)) hide)
     )
@@
       (effects (font (size 1.27 1.27)) hide)
     )
+    (property "Manufacturer_Part_Number" "dnp" (at 30.48 85.09 0)
+      (effects (font (size 1.27 1.27)) hide)
+    )
     (pin "1")
     (instances
@@
     )
     (property "Datasheet" "http://infocenter.arm.com/help/topic/com.arm.doc.ddi0314h/DDI0314H_coresight_components_trm.pdf" (at 25.4 163.83 90)
+      (effects (font (size 1.27 1.27)) hide)
+    )
+    (property "Manufacturer_Part_Number" "M50-3500542" (at 34.29 132.08 0)
       (effects (font (size 1.27 1.27)) hide)
     )
@@
       (effects (font (size 1.27 1.27)) hide)
     )
+    (property "Manufacturer_Part_Number" "JMK107ABJ106MA-T " (at 66.04 39.37 0)
+      (effects (font (size 1.27 1.27)) hide)
+    )
     (pin "1")
     (pin "2")
@@
       (effects (font (size 1.27 1.27)) hide)
     )
+    (property "Manufacturer_Part_Number" "LQM18PN2R2MGHD" (at 38.1 21.59 0)
+      (effects (font (size 1.27 1.27)) hide)
+    )

Commit message: part #s
Parts:
- J4: Manufacturer_Part_Number 73412-0110 -> U.FL-R-SMT-1(10)
Changed lines of the file:
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@@
       (effects (font (size 1.27 1.27)) hide)
     )
-    (property "Manufacturer_Part_Number" "73412-0110" (at 274.32 92.71 0)
+    (property "Manufacturer_Part_Number" "U.FL-R-SMT-1(10)" (at 274.32 92.71 0)
       (effects (font (size 1.27 1.27)) hide)
     )

Commit message: exports
Parts:
- J2, J3: value Conn_01x01 -> ~
Other:
- note added: "Measure V_BATT on ADC"
- note added: "Solder 3V non-rechargable cell (CR2)"
Changed lines of the file:
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@@
     (stroke (width 0) (type default))
+  )
+  (text "Solder 3V non-rechargable cell (CR2)" (at 13.97 82.55 0)
+    (effects (font (size 1.27 1.27)) (justify left bottom))
+  )
+  (text "Measure V_BATT on ADC" (at 146.05 151.13 0)
+    (effects (font (size 1.27 1.27)) (justify left bottom))
   )
   (label "SENS_SPI_CS" (at 210.82 149.86 0) (fields_autoplaced)
@@
   )
   (symbol (lib_id "Connector_Generic:Conn_01x01") (at 30.48 78.74 270) (unit 1)
-    (in_bom no) (on_board yes) (dnp no) (fields_autoplaced)
-    (property "Reference" "J2" (at 33.02 78.105 90)
-      (effects (font (size 1.27 1.27)) (justify left))
-    )
-    (property "Value" "Conn_01x01" (at 33.02 80.645 90)
+    (in_bom no) (on_board yes) (dnp no)
+    (property "Reference" "J2" (at 33.02 78.74 90)
+      (effects (font (size 1.27 1.27)) (justify left))
+    )
+    (property "Value" "~" (at 33.02 78.74 90)
       (effects (font (size 1.27 1.27)) (justify left))
     )
@@
   (symbol (lib_id "Connector_Generic:Conn_01x01") (at 30.48 85.09 90) (unit 1)
     (in_bom no) (on_board yes) (dnp no) (fields_autoplaced)
-    (property "Reference" "J3" (at 33.02 84.455 90)
+    (property "Reference" "J3" (at 33.02 85.725 90)
       (effects (font (size 1.27 1.27)) (justify right))
     )
-    (property "Value" "Conn_01x01" (at 33.02 86.995 90)
+    (property "Value" "~" (at 33.02 86.995 90)
       (effects (font (size 1.27 1.27)) (justify right))
     )

Commit message: gnss_uart
Parts:
- removed R3, R4: 10k, Resistor_SMD:R_0603_1608Metric, symbol Device:R_Small
Connections:
- net GNSS_TX: now reaches U2.39 (PTB16)
- net GNSS_TX: now also U3.25 (TXD1)
- net GNSS_RX: now reaches U2.40 (PTB17)
- net GNSS_RX: now also U3.26 (RXD1)
- net GNSS_I2C_SCL: no longer names the net of U2.44 (PTC1/LLWU_P6/RTC_CLKIN)
- net GNSS_I2C_SCL: no longer U3.6 (I2C_SCL)
- net GNSS_I2C_SDA: no longer names the net of U2.45 (PTC2)
- net GNSS_I2C_SDA: no longer U3.3 (I2C_SDA)
Other:
- moved on the sheet: C20, R5
